File: PMS.kicad_pcb (KiCad board)
At the start: 2 copper layers, 175.5 x 87 mm, 178 parts, among them IC2 SI4459ADY-T1-GE3, IC8 SI4485DY-T1-GE3, J1 XT60-M, J10 XT60-M, J11 CONN_06SILK_FEMALE_PTH, J12 CONN_06SILK_FEMALE_PTH, J13 CONN_06SILK_FEMALE_PTH, J2 XT60-M, J3 Vertical Qwiic Connector, J4 UJ2-MIBH-2-SMT-TR-67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

Commit message: Add Mounting Holes
Parts:
- added ?: , , F.Cu at (233.5, 61.0)
- added ?: , , F.Cu at (67.0, 61.0)
- added ?: , , F.Cu at (233.5, 139.0)
- added ?: , , F.Cu at (67.0, 139.0)
